File: thermidity-kicad/thermidity.kicad_pcb (KiCad board)
At the start: 2 copper layers, 60 x 30 mm, 18 parts, among them J1 Battery, J2 Display, J3 ISP, U1 ATmega328P, U2 HIH-5030, U3 TMP36

Commit message: remove the 1pF capacitor between AREF and GND
- takes ~125us to discharge after switching from AVCC to internal 1.1 voltage reference and for the reference to settle
- shouldn't be necessary and hopefully the 16x oversampling benefits from some noise
- one part less
Parts:
- removed the C3 at (136.4, 73.7)
- renumbered C2 to C1, C6 to C2, C5 to C3, R3 to R1, R4 to R2, R5 to R3
Connections:
- U1 pad 20: Net-(U1-Pad20) -> unconnected-(U1-Pad20)
Routing:
- net Net-(U1-Pad20): track 3.27 -> 0.00 mm
- net GND: track 20.7 -> 19.2 mm, vias 8 -> 7

Commit message: Ratiometric measurement of temperature with a thermistor (#18)
- replace TMP36 with a thermistor NTC 100k
- put back 1nF cap between AREF and GND
- wait 150us for the cap to discharge before converting with 1.1V reference
- uint16_t is enough for 16x ADC
- SMD footprint instead of TH for thermistor
- calculate temperature
- rounding of temperature compensated relative humidity
- no need for battery voltage in mV
Parts:
- removed the C3 at (135.2, 84.8)
- removed U3: TMP36, TMP36GT9:XDCR_TMP36GT9
- added C2: 1nF, Capacitor_SMD:C_1206_3216Metric_Pad1.33x1.80mm_HandSolder, F.Cu at (136.3, 73.6)
- added R3: 100k, Resistor_SMD:R_0805_2012Metric_Pad1.20x1.40mm_HandSolder, F.Cu at (143.7, 84.9)
- added TH1: NTC 100k, Resistor_SMD:R_0805_2012Metric_Pad1.20x1.40mm_HandSolder, F.Cu at (138.4, 84.9)
- R1: value 1M -> 300K
- R2: value 1M -> 1.2M
- moved R4 0.30 mm to (148.9, 84.9)
- renumbered C2 to C3, R3 to R4
Routing:
- net unconnected-(U1-Pad20): track 0.00 -> 3.28 mm
- net Net-(R2-Pad1): track 28.5 -> 26.4 mm
- net Net-(U1-Pad25): track 8.09 -> 9.96 mm
- net GND: track 19.2 -> 20.5 mm
- net Net-(R4-Pad1): track 13.0 -> 13.7 mm

Commit message: update README and schematic + PCB
Parts:
- R3: value 100k -> 100k 0.1%
- TH1: value NTC 100k -> NTC 100k 0.1°C
Changed lines of the file:
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@@
       (effects (font (size 1 1) (thickness 0.15)))
     )
-    (fp_text value "NTC 100k" (at 0 1.65) (layer "F.Fab")
+    (fp_text value "NTC 100k 0.1°C" (at 0 1.65) (layer "F.Fab")
       (effects (font (size 1 1) (thickness 0.15)))
     )
@@
       (effects (font (size 1 1) (thickness 0.15)))
     )
-    (fp_text value "100k" (at 0 1.65) (layer "F.Fab")
-      (effects (font (size 1 1) (thickness 0.15)))
-    )
+    (fp_text value "100k 0.1%" (at 0 1.65) (layer "F.Fab")
+      (effects (font (size 1 1) (thickness 0.15)))
+    )
